Commit message: 源码

File: xarm_ros/xarm_description/urdf/dual_xarm6_robot.urdf.xacro (robot description, xacro)
@@ -6,5 +6,5 @@
   <xacro:arg name="limited" default="false"/>
   <xacro:arg name="effort_control" default="false"/>
-  <xacro:arg name="add_gripper" default="true"/>
+  <xacro:arg name="add_gripper" default="false"/>
   <xacro:include filename="$(find xarm_description)/urdf/xarm6_robot_macro.xacro" />
   <xacro:include filename="$(find xarm_gripper)/urdf/xarm_gripper_model.xacro" />
@@ -12,55 +12,12 @@
   <link name="ground" />
   <!-- launch left arm -->
-  <xacro:xarm6_robot prefix="$(arg prefix_1)" namespace="$(arg ros_namespace)" limited="$(arg limited)" attach_to="ground" xyz="-0.5 0.09916 0" rpy="-1.57 0 -0.349"/>
+  <xacro:xarm6_robot prefix="$(arg prefix_1)" namespace="$(arg ros_namespace)" limited="$(arg limited)" attach_to="ground" xyz="0 0 0" rpy="0 0 0"/>
   <xacro:if value="$(arg add_gripper)">
-    <xacro:load_gripper prefix="$(arg prefix_1)" attach_to="$(arg prefix_1)link6" />
+    <xacro:load_gripper attach_to="$(arg prefix_1)link6" />
   </xacro:if>
   <!-- launch right arm -->
-  <xacro:xarm6_robot prefix="$(arg prefix_2)" namespace="$(arg ros_namespace)" limited="$(arg limited)" attach_to="ground" xyz="-0.5 -0.09916 0" rpy="1.57 0 0.349"/>
+  <xacro:xarm6_robot prefix="$(arg prefix_2)" namespace="$(arg ros_namespace)" limited="$(arg limited)" attach_to="ground" xyz="0 1 0" rpy="0 0 0"/>
   <xacro:if value="$(arg add_gripper)">
-    <xacro:load_gripper prefix="$(arg prefix_2)" attach_to="$(arg prefix_2)link6" />
+    <xacro:load_gripper attach_to="$(arg prefix_2)link6" />
   </xacro:if>
-  <!-- add body link -->
-  <link name="body">
-  <inertial>
-    <origin xyz="0.079038 -0.38069 -0.076812" rpy="0 0 0" />
-    <mass
-      value="20.22" />
-    <inertia
-      ixx="1.6025"
-      ixy="0.038852"
-      ixz="0.0033194"
-      iyy="0.71269"
-      iyz="0.014666"
-      izz="1.5939" />
-  </inertial>
-  <visual>
-    <origin
-      xyz="-0.5 -0.09916 0"
-      rpy="1.57 0 0.349" />
-    <geometry>
-      <mesh
-        filename="package://xarm_planner/meshes/body.stl" />
-    </geometry>
-    <material
-      name="">
-      <color
-        rgba="1.0 1.0 1.0 1.0" />
-    </material>
-  </visual>
-  <collision>
-    <origin
-      xyz="-0.5 -0.09916 0"
-      rpy="1.57 0 0.349" />
-    <geometry>
-      <mesh
-        filename="package://xarm_planner/meshes/body.stl" />
-    </geometry>
-  </collision>
-</link>
-<joint name="ground_joint" type="fixed">
-    <parent link="ground" />
-    <child link = "body" />
-    <origin xyz="0 0 0" rpy="0 0 0" />
-</joint>
 </robot>

File: xarm_ros/xarm_gripper/urdf/xarm_gripper.urdf.xacro (robot description, xacro)
@@ -280,5 +280,5 @@
       effort="50"
       velocity="2" />
-    <mimic joint="${prefix}drive_joint" multiplier="1" offset="0" />
+    <mimic joint="drive_joint" multiplier="1" offset="0" />
   </joint>
   <link

Commit message: 源码

File: xarm_ros/xarm_description/urdf/dual_xarm6_robot.urdf.xacro (robot description, xacro)
@@ -6,5 +6,5 @@
   <xacro:arg name="limited" default="false"/>
   <xacro:arg name="effort_control" default="false"/>
-  <xacro:arg name="add_gripper" default="false"/>
+  <xacro:arg name="add_gripper" default="true"/>
   <xacro:include filename="$(find xarm_description)/urdf/xarm6_robot_macro.xacro" />
   <xacro:include filename="$(find xarm_gripper)/urdf/xarm_gripper_model.xacro" />
@@ -12,12 +12,55 @@
   <link name="ground" />
   <!-- launch left arm -->
-  <xacro:xarm6_robot prefix="$(arg prefix_1)" namespace="$(arg ros_namespace)" limited="$(arg limited)" attach_to="ground" xyz="0 0 0" rpy="0 0 0"/>
+  <xacro:xarm6_robot prefix="$(arg prefix_1)" namespace="$(arg ros_namespace)" limited="$(arg limited)" attach_to="ground" xyz="-0.5 0.09916 0" rpy="-1.57 0 -0.349"/>
   <xacro:if value="$(arg add_gripper)">
-    <xacro:load_gripper attach_to="$(arg prefix_1)link6" />
+    <xacro:load_gripper prefix="$(arg prefix_1)" attach_to="$(arg prefix_1)link6" />
   </xacro:if>
   <!-- launch right arm -->
-  <xacro:xarm6_robot prefix="$(arg prefix_2)" namespace="$(arg ros_namespace)" limited="$(arg limited)" attach_to="ground" xyz="0 1 0" rpy="0 0 0"/>
+  <xacro:xarm6_robot prefix="$(arg prefix_2)" namespace="$(arg ros_namespace)" limited="$(arg limited)" attach_to="ground" xyz="-0.5 -0.09916 0" rpy="1.57 0 0.349"/>
   <xacro:if value="$(arg add_gripper)">
-    <xacro:load_gripper attach_to="$(arg prefix_2)link6" />
+    <xacro:load_gripper prefix="$(arg prefix_2)" attach_to="$(arg prefix_2)link6" />
   </xacro:if>
+  <!-- add body link -->
+  <link name="body">
+  <inertial>
+    <origin xyz="0.079038 -0.38069 -0.076812" rpy="0 0 0" />
+    <mass
+      value="20.22" />
+    <inertia
+      ixx="1.6025"
+      ixy="0.038852"
+      ixz="0.0033194"
+      iyy="0.71269"
+      iyz="0.014666"
+      izz="1.5939" />
+  </inertial>
+  <visual>
+    <origin
+      xyz="-0.5 -0.09916 0"
+      rpy="1.57 0 0.349" />
+    <geometry>
+      <mesh
+        filename="package://xarm_planner/meshes/body.stl" />
+    </geometry>
+    <material
+      name="">
+      <color
+        rgba="1.0 1.0 1.0 1.0" />
+    </material>
+  </visual>
+  <collision>
+    <origin
+      xyz="-0.5 -0.09916 0"
+      rpy="1.57 0 0.349" />
+    <geometry>
+      <mesh
+        filename="package://xarm_planner/meshes/body.stl" />
+    </geometry>
+  </collision>
+</link>
+<joint name="ground_joint" type="fixed">
+    <parent link="ground" />
+    <child link = "body" />
+    <origin xyz="0 0 0" rpy="0 0 0" />
+</joint>
 </robot>

Commit message: 机器人模型添加底盘，修改手臂位置，使gazebo稳定

File: xarm_ros/xarm_description/urdf/dual_xarm6_robot.urdf.xacro (robot description, xacro)
@@ -11,12 +11,12 @@
   <xacro:include filename="$(find xarm_description)/urdf/common.gazebo.xacro" />
   <!-- ground instead of world, for the arms to attach -->
-  <link name="ground" />
+  <!--<link name="ground" />-->
   <!-- launch left arm -->
-  <xacro:xarm6_robot prefix="$(arg prefix_1)" namespace="$(arg ros_namespace)" limited="$(arg limited)" attach_to="ground" xyz="-0.5 0.09916 0" rpy="-1.57 0 -0.349"/>
+  <xacro:xarm6_robot prefix="$(arg prefix_1)" namespace="$(arg ros_namespace)" limited="$(arg limited)" attach_to="bottom_link" xyz="-0.5 0.09916 1" rpy="-1.57 0 -0.049"/>
   <xacro:if value="$(arg add_gripper)">
     <xacro:load_gripper prefix="$(arg prefix_1)" attach_to="$(arg prefix_1)link6" />
   </xacro:if>
   <!-- launch right arm -->
-  <xacro:xarm6_robot prefix="$(arg prefix_2)" namespace="$(arg ros_namespace)" limited="$(arg limited)" attach_to="ground" xyz="-0.5 -0.09916 0" rpy="1.57 0 0.349"/>
+  <xacro:xarm6_robot prefix="$(arg prefix_2)" namespace="$(arg ros_namespace)" limited="$(arg limited)" attach_to="bottom_link" xyz="-0.5 -0.09916 1" rpy="1.57 0 0.049"/>
   <xacro:if value="$(arg add_gripper)">
     <xacro:load_gripper prefix="$(arg prefix_2)" attach_to="$(arg prefix_2)link6" />
@@ -67,8 +67,37 @@
   </collision>
 </link>
-<joint name="ground_joint" type="fixed">
-    <parent link="ground" />
+<joint name="bottom_joint" type="fixed">
+    <parent link="bottom_link" />
     <child link = "body" />
-    <origin xyz="0 0 0" rpy="0 0 0" />
+    <origin xyz="0 0 1" rpy="0 0 0" />
 </joint>
+    <link name="bottom_link">
+	   <inertial>
+		  <origin
+		    xyz="0 0 0"
+		    rpy="0 0 0" />
+		  <mass
+		    value="444.11" />
+		  <inertia
+		    ixx="337.5"
+		    ixy="3.3871E-16"
+		    ixz="-3.6082E-14"
+		    iyy="674.82"
+		    iyz="1.3219E-17"
+		    izz="337.5" />
+		</inertial>
+        <visual>
+              <origin xyz=" 0 0 0"  rpy="0 0 0"/>
+                  <geometry>
+                       <box size="20 20 0.02" />
+                  </geometry>
+              <material name="Hide" />
+        </visual>
+        <collision>
+            <origin xyz=" 0 0 0"  rpy="0 0 0"/>
+            <geometry>
+                <box size="20 20 0.05" />
+            </geometry>
+        </collision>
+    </link>
 </robot>

Commit message: 添加甲爪在gazebo内的插件，使模型稳定

File: xarm_ros/xarm_description/urdf/dual_xarm6_robot.urdf.xacro (robot description, xacro)
@@ -15,10 +15,10 @@
   <xacro:xarm6_robot prefix="$(arg prefix_1)" namespace="$(arg ros_namespace)" limited="$(arg limited)" attach_to="bottom_link" xyz="-0.5 0.09916 1" rpy="-1.57 0 -0.049"/>
   <xacro:if value="$(arg add_gripper)">
-    <xacro:load_gripper prefix="$(arg prefix_1)" attach_to="$(arg prefix_1)link6" />
+    <xacro:load_gripper prefix="$(arg prefix_1)" attach_to="$(arg prefix_1)link6" rpy="0 0 0" xyz="0 0 0"/>
   </xacro:if>
   <!-- launch right arm -->
   <xacro:xarm6_robot prefix="$(arg prefix_2)" namespace="$(arg ros_namespace)" limited="$(arg limited)" attach_to="bottom_link" xyz="-0.5 -0.09916 1" rpy="1.57 0 0.049"/>
   <xacro:if value="$(arg add_gripper)">
-    <xacro:load_gripper prefix="$(arg prefix_2)" attach_to="$(arg prefix_2)link6" />
+    <xacro:load_gripper prefix="$(arg prefix_2)" attach_to="$(arg prefix_2)link6" rpy="0 0 0" xyz="0 0 0"/>
   </xacro:if>
   <gazebo>

File: xarm_ros/xarm_gripper/urdf/xarm_gripper.gazebo.xacro (robot description, xacro)
@@ -4,5 +4,5 @@
   <xacro:macro name="mimic_joint_plugin_gazebo" params="name_prefix following_joint mimic_joint has_pid:=false multiplier:=1.0 offset:=0 sensitiveness:=0.0 max_effort:=1.0 robot_namespace:=''">
     <gazebo>
-      <plugin name="${name_prefix}mimic_joint_plugin" filename="libroboticsgroup_gazebo_mimic_joint_plugin.so">
+      <plugin name="${name_prefix}mimic_joint_plugin" filename="libroboticsgroup_upatras_gazebo_mimic_joint_plugin.so">
         <joint>${following_joint}</joint>
         <mimicJoint>${mimic_joint}</mimicJoint>

File: xarm_ros/xarm_gripper/urdf/xarm_gripper.xacro (robot description, xacro)
@@ -2,4 +2,33 @@
 <robot xmlns:xacro="http://ros.org/wiki/xacro" name="xarm_gripper">
   <xacro:include filename="$(find xarm_gripper)/urdf/xarm_gripper_model.xacro" />
-  <xacro:load_gripper />
+<link name="bottom_link">
+	   <inertial>
+		  <origin
+		    xyz="0 0 0"
+		    rpy="0 0 0" />
+		  <mass
+		    value="444.11" />
+		  <inertia
+		    ixx="337.5"
+		    ixy="3.3871E-16"
+		    ixz="-3.6082E-14"
+		    iyy="674.82"
+		    iyz="1.3219E-17"
+		    izz="337.5" />
+		</inertial>
+        <visual>
+              <origin xyz=" 0 0 0"  rpy="0 0 0"/>
+                  <geometry>
+                       <box size="20 20 0.02" />
+                  </geometry>
+              <material name="Hide" />
+        </visual>
+        <collision>
+            <origin xyz=" 0 0 0"  rpy="0 0 0"/>
+            <geometry>
+                <box size="20 20 0.05" />
+            </geometry>
+        </collision>
+    </link>
+  <xacro:load_gripper attach_to="bottom_link" rpy="0 0 0" xyz="0 0 1"/>
 </robot>

File: xarm_ros/xarm_gripper/urdf/xarm_gripper_model.xacro (robot description, xacro)
@@ -12,27 +12,22 @@
     <!-- <xacro:gazebo_ros_control_plugin namespace="${ns}"/> -->
     <xacro:xarm_gripper_urdf prefix="${prefix}" attach_to="${attach_to}" xyz="${xyz}" rpy="${rpy}" />
-    <xacro:if value="${effort_control}">
-      <xacro:xarm_gripper_transmission prefix="${prefix}" hard_interface="EffortJointInterface" />
-    </xacro:if>
-    <xacro:unless value="${effort_control}">
-      <xacro:xarm_gripper_transmission prefix="${prefix}" hard_interface="PositionJointInterface" />
-    </xacro:unless>
+    <xacro:xarm_gripper_transmission prefix="${prefix}" hard_interface="PositionJointInterface" />
     <xacro:xarm_gripper_gazebo prefix="${prefix}" />
     <!-- mimic_joint_plugin has to be installed: -->
-    <xacro:mimic_joint_plugin_gazebo name_prefix="left_finger_joint"
-    following_joint="drive_joint" mimic_joint="left_finger_joint"
-    has_pid="true" multiplier="1.0" max_effort="10.0" />
-    <xacro:mimic_joint_plugin_gazebo name_prefix="left_inner_knuckle_joint"
-    following_joint="drive_joint" mimic_joint="left_inner_knuckle_joint"
-    has_pid="true" multiplier="1.0" max_effort="10.0" />
-    <xacro:mimic_joint_plugin_gazebo name_prefix="right_outer_knuckle_joint"
-    following_joint="drive_joint" mimic_joint="right_outer_knuckle_joint"
-    has_pid="true" multiplier="1.0" max_effort="10.0" />
-    <xacro:mimic_joint_plugin_gazebo name_prefix="right_finger_joint"
-    following_joint="drive_joint" mimic_joint="right_finger_joint"
-    has_pid="true" multiplier="1.0" max_effort="10.0" />
-    <xacro:mimic_joint_plugin_gazebo name_prefix="right_inner_knuckle_joint"
-    following_joint="drive_joint" mimic_joint="right_inner_knuckle_joint"
-    has_pid="true" multiplier="1.0" max_effort="10.0" />
+    <xacro:mimic_joint_plugin_gazebo name_prefix="${prefix}left_finger_joint"
+    following_joint="${prefix}drive_joint" mimic_joint="${prefix}left_finger_joint"
+    has_pid="false" multiplier="1.0" max_effort="10.0" />
+    <xacro:mimic_joint_plugin_gazebo name_prefix="${prefix}left_inner_knuckle_joint"
+    following_joint="${prefix}drive_joint" mimic_joint="${prefix}left_inner_knuckle_joint"
+    has_pid="false" multiplier="1.0" max_effort="10.0" />
+    <xacro:mimic_joint_plugin_gazebo name_prefix="${prefix}right_outer_knuckle_joint"
+    following_joint="${prefix}drive_joint" mimic_joint="${prefix}right_outer_knuckle_joint"
+    has_pid="false" multiplier="1.0" max_effort="10.0" />
+    <xacro:mimic_joint_plugin_gazebo name_prefix="${prefix}right_finger_joint"
+    following_joint="${prefix}drive_joint" mimic_joint="${prefix}right_finger_joint"
+    has_pid="false" multiplier="1.0" max_effort="10.0" />
+    <xacro:mimic_joint_plugin_gazebo name_prefix="${prefix}right_inner_knuckle_joint"
+    following_joint="${prefix}drive_joint" mimic_joint="${prefix}right_inner_knuckle_joint"
+    has_pid="false" multiplier="1.0" max_effort="10.0" />
   </xacro:macro>
 </robot>
